File: hardware/kicad/snopf.kicad_pcb (KiCad board)
At the start: 2 copper layers, 14 x 17.3 mm, 18 parts, among them J1 USB_A, SW1 User Button, U1 ATTINY85-20SU, Y1 12 MHz

Commit message: Add a 3D printable casing
Parts:
- SW1: footprint Button_Switch_SMD:SW_SPST_EVQQ2 -> snopf_footprints:SW_SPST_EVQQ2
